File: Connectors.kicad_sch (KiCad schematic)
At the start: 22 parts, among them J1 CAN, J2 USART, J3 2171750001, J401 SWD, U2 ICM-42688-P, U6 TJA1051T/3

Commit message: add mounting hole
Parts:
- removed C29: 100n, Capacitor_SMD:C_0603_1608Metric, symbol Device:C
- removed C7: 2u2, Capacitor_SMD:C_0603_1608Metric, symbol Device:C_Small
- added C2: 100n, Capacitor_SMD:C_0402_1005Metric, symbol Device:C_Small
- added C4: 2u2, Capacitor_SMD:C_0603_1608Metric, symbol Device:C_Small
- J1: value CAN -> KH-1.27PH180-1X4P-L7.2; footprint Connector_PinHeader_1.00mm:PinHeader_1x04_P1.00mm_Vertical_SMD_Pin1Right -> Connector_PinHeader_1.27mm:PinHeader_1x04_P1.27mm_Vertical
- J2: value USART -> KH-1.27PH180-1X4P-L7.2; footprint Connector_PinHeader_1.00mm:PinHeader_1x04_P1.00mm_Vertical_SMD_Pin1Right -> Connector_PinHeader_1.27mm:PinHeader_1x04_P1.27mm_Vertical
- J401: value SWD -> B3U-3000P-B; footprint Connector_PinHeader_1.27mm:PinHeader_2x05_P1.27mm_Vertical_SMD -> Connector_PinHeader_1.27mm:PinHeader_2x05_P1.27mm_Vertical
- R19, R20: footprint Resistor_SMD:R_0603_1608Metric -> Resistor_SMD:R_0402_1005Metric
Connections:
- net +3.3V: now also C4.1
- net +5V: now also C2.1
- net GND: now also C2.2, C4.2
Changed lines of the file:
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@@
 	(wire
 		(pts
-			(xy 80.01 49.53) (xy 80.01 50.8)
+			(xy 80.01 46.99) (xy 80.01 50.8)
 		)
 		(stroke
@@
 			)
 		)
-		(property "Value" "SWD"
+		(property "Value" "B3U-3000P-B"
 			(at 50.8 135.89 0)
 			(effects
@@
 					(size 1.27 1.27)
 				)
+				(hide yes)
 			)
 		)
-		(property "Footprint" "Connector_PinHeader_1.27mm:PinHeader_2x05_P1.27mm_Vertical_SMD"
+		(property "Footprint" "Connector_PinHeader_1.27mm:PinHeader_2x05_P1.27mm_Vertical"
 			(at 49.53 128.27 0)
 			(effects
@@
 	)
 	(symbol
-		(lib_id "Device:R")
-		(at 85.09 74.93 0)
+		(lib_id "Device:C_Small")
+		(at 220.98 107.95 0)
 		(unit 1)
 		(exclude_from_sim no)
@@
 		(on_board yes)
 		(dnp no)
-		(property "Reference" "R19"
-			(at 86.614 73.66 0)
+		(property "Reference" "C4"
+			(at 223.52 106.68 0)
 			(effects
 				(font
@@
 			)
 		)
-		(property "Value" "60R"
-			(at 86.614 76.2 0)
+		(property "Value" "2u2"
+			(at 223.52 109.22 0)
 			(effects
 				(font
@@
 			)
 		)
-		(property "Footprint" "Resistor_SMD:R_0603_1608Metric"
-			(at 83.312 74.93 90)
+		(property "Footprint" "Capacitor_SMD:C_0603_1608Metric"
+			(at 220.98 107.95 0)
 			(effects
 				(font
@@
 		)
 		(property "Datasheet" "~"
-			(at 85.09 74.93 0)
+			(at 220.98 107.95 0)
 			(effects
 				(font
@@
 			)
 		)
-		(property "Description" "Resistor"
-			(at 85.09 74.93 0)
+		(property "Description" ""
+			(at 220.98 107.95 0)
 			(effects
 				(font
 					(size 1.27 1.27)
 				)
-				(hide yes)
 			)
 		)
-		(pin "2"
+		(property "LCSC Part #" "C23630"
+			(at 220.98 107.95 0)
+			(effects
+				(font
+					(size 1.27 1.27)
+				)
+				(hide yes)
+			)
 		)
 		(pin "1"
 		)
+		(pin "2"
+		)
 		(instances
 			(project "MX_IMU"
 				(path "/8ed38441-7d4e-4e89-870f-07e11c6dce38/3e6b1080-2480-49a7-8bae-2dbfae5f98f5"
-					(reference "R19")
+					(reference "C4")
 					(unit 1)
 				)
@@
 	)
 	(symbol
-		(lib_id "Device:C")
-		(at 80.01 45.72 0)
+		(lib_id "Device:R")
+		(at 85.09 74.93 0)
 		(unit 1)
 		(exclude_from_sim no)
@@
 		(on_board yes)
 		(dnp no)
-		(property "Reference" "C29"
-			(at 82.55 44.45 0)
+		(property "Reference" "R19"
+			(at 86.614 73.66 0)
 			(effects
 				(font
@@
 			)
 		)
-		(property "Value" "100n"
-			(at 82.55 46.99 0)
+		(property "Value" "60R"
+			(at 86.614 76.2 0)
 			(effects
 				(font
@@
 			)
 		)
-		(property "Footprint" "Capacitor_SMD:C_0603_1608Metric"
-			(at 80.9752 49.53 0)
+		(property "Footprint" "Resistor_SMD:R_0402_1005Metric"
+			(at 83.312 74.93 90)
 			(effects
 				(font
@@
 		)
 		(property "Datasheet" "~"
-			(at 80.01 45.72 0)
+			(at 85.09 74.93 0)
 			(effects
 				(font
@@
 			)
 		)
-		(property "Description" "Unpolarized capacitor"
-			(at 80.01 45.72 0)
+		(property "Description" "Resistor"
+			(at 85.09 74.93 0)
 			(effects
 				(font
@@
 			)
 		)
-		(pin "1"
-		)
 		(pin "2"
 		)
+		(pin "1"
+		)
 		(instances
 			(project "MX_IMU"
 				(path "/8ed38441-7d4e-4e89-870f-07e11c6dce38/3e6b1080-2480-49a7-8bae-2dbfae5f98f5"
-					(reference "C29")
+					(reference "R19")
 					(unit 1)
 				)
@@
 			)
 		)
-		(property "Value" "CAN"
+		(property "Value" "KH-1.27PH180-1X4P-L7.2"
 			(at 144.78 69.85 0)
 			(effects
@@
 				)
 				(justify right)
+				(hide yes)
 			)
 		)
-		(property "Footprint" "Connector_PinHeader_1.00mm:PinHeader_1x04_P1.00mm_Vertical_SMD_Pin1Right"
+		(property "Footprint" "Connector_PinHeader_1.27mm:PinHeader_1x04_P1.27mm_Vertical"
 			(at 143.51 67.31 0)
 			(effects
@@
 			)
 		)
-		(property "Footprint" "Resistor_SMD:R_0603_1608Metric"
+		(property "Footprint" "Resistor_SMD:R_0402_1005Metric"
 			(at 93.472 74.93 90)
 			(effects
@@
 	)
 	(symbol
-		(lib_id "Device:C_Small")
-		(at 220.98 107.95 0)
+		(lib_id "Connector:Conn_01x04_Pin")
+		(at 143.51 54.61 0)
+		(mirror y)
 		(unit 1)
 		(exclude_from_sim no)
@@
 		(on_board yes)
 		(dnp no)
-		(fields_autoplaced yes)
-		(property "Reference" "C7"
-			(at 223.52 106.6862 0)
+		(property "Reference" "J2"
+			(at 144.78 54.61 0)
 			(effects
 				(font
 					(size 1.27 1.27)
 				)
-				(justify left)
+				(justify right)
 			)
 		)
-		(property "Value" "2u2"
-			(at 223.52 109.2262 0)
+		(property "Value" "KH-1.27PH180-1X4P-L7.2"
+			(at 144.78 57.15 0)
 			(effects
 				(font
 					(size 1.27 1.27)
 				)
-				(justify left)
+				(justify right)
+				(hide yes)
 			)
 		)
-		(property "Footprint" "Capacitor_SMD:C_0603_1608Metric"
-			(at 220.98 107.95 0)
+		(property "Footprint" "Connector_PinHeader_1.27mm:PinHeader_1x04_P1.27mm_Vertical"
+			(at 143.51 54.61 0)
 			(effects
 				(font
@@
 		)
 		(property "Datasheet" "~"
-			(at 220.98 107.95 0)
+			(at 143.51 54.61 0)
 			(effects
 				(font
@@
 		)
 		(property "Description" ""
-			(at 220.98 107.95 0)
+			(at 143.51 54.61 0)
 			(effects
 				(font
@@
 		(pin "2"
 		)
+		(pin "3"
+		)
+		(pin "4"
+		)
 		(instances
 			(project "MX_IMU"
 				(path "/8ed38441-7d4e-4e89-870f-07e11c6dce38/3e6b1080-2480-49a7-8bae-2dbfae5f98f5"
-					(reference "C7")
+					(reference "J2")
 					(unit 1)
 				)
@@
 	)
 	(symbol
-		(lib_id "Connector:Conn_01x04_Pin")
-		(at 143.51 54.61 0)
-		(mirror y)
+		(lib_id "Device:C_Small")
+		(at 80.01 44.45 0)
 		(unit 1)
 		(exclude_from_sim no)
@@
 		(on_board yes)
 		(dnp no)
-		(property "Reference" "J2"
-			(at 144.78 54.61 0)
+		(property "Reference" "C2"
+			(at 82.55 43.18 0)
 			(effects
 				(font
 					(size 1.27 1.27)
 				)
-				(justify right)
+				(justify left)
 			)
 		)
-		(property "Value" "USART"
-			(at 144.78 57.15 0)
+		(property "Value" "100n"
+			(at 82.55 45.72 0)
 			(effects
 				(font
 					(size 1.27 1.27)
 				)
-				(justify right)
+				(justify left)
 			)
 		)
-		(property "Footprint" "Connector_PinHeader_1.00mm:PinHeader_1x04_P1.00mm_Vertical_SMD_Pin1Right"
-			(at 143.51 54.61 0)
+		(property "Footprint" "Capacitor_SMD:C_0402_1005Metric"
+			(at 80.01 44.45 0)
 			(effects
 				(font
@@
 		)
 		(property "Datasheet" "~"
-			(at 143.51 54.61 0)
+			(at 80.01 44.45 0)
 			(effects
 				(font
@@
 		)
 		(property "Description" ""
-			(at 143.51 54.61 0)
+			(at 80.01 44.45 0)
 			(effects
 				(font
@@
 			)
 		)
-		(pin "1"
+		(property "LCSC Part #" "C1525"
+			(at 80.01 44.45 0)
+			(effects
+				(font
+					(size 1.27 1.27)
+				)
+				(hide yes)
+			)
 		)
 		(pin "2"
 		)
-		(pin "3"
-		)
-		(pin "4"
+		(pin "1"
 		)
 		(instances
 			(project "MX_IMU"
 				(path "/8ed38441-7d4e-4e89-870f-07e11c6dce38/3e6b1080-2480-49a7-8bae-2dbfae5f98f5"
-					(reference "J2")
+					(reference "C2")
 					(unit 1)
 				)
