File: MX_IMU.kicad_pcb (KiCad board)
At the start: 4 copper layers, 40 x 36 mm, 55 parts, among them J1 KH-1.27PH180-1X4P-L7.2, J2 KH-1.27PH180-1X4P-L7.2, J3 2171750001, J4 ZX-PZ2.54-1-5PZZ, SW1 SW_SPST, U1 ld39150dt33-r, U2 ICM-42688-P, U200 STM32F405RGT6, U4 AT24C256, U6 TJA1051T/3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

Commit message: add coper ground and other design
Parts:
- moved C210 1.10 mm to (126.2, 98.9)
- moved C211 1.10 mm to (126.2, 104.9)
- moved Y200 1.10 mm to (126.2, 101.9)
- moved R200 0.59 mm to (129.9, 102.5)
- moved C206 0.25 mm to (129.6, 105.4)
Routing:
- net /Connectors/CAN1-: track 11.0 -> 12.4 mm
- net GND: track 81.7 -> 83.0 mm, vias 48 -> 67
- net HSE_IN: track 7.88 -> 8.98 mm
- net Net-(C211-Pad1): track 3.07 -> 4.02 mm
- net Net-(J2-Pin_3): track 4.73 -> 5.37 mm
- added copper zone on B.Cu, net GND
- added copper zone on F.Cu, net GND
Other:
- board text added: "IMU_Ver_1.0 by MX Motion July,2025"
- board text removed: "IMU_Ver_1.0 by MX Motion Canada Day"

Commit message: Version for JLCPCB
Parts:
- C10: footprint Capacitor_SMD:C_0201_0603Metric -> Capacitor_SMD:C_0402_1005Metric
- moved C10 0.16 mm to (145.8, 115.8)
Routing:
- net GND: vias 67 -> 76
Changed lines of the file:
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@@
 		(6 "In2.Cu" signal)
 		(2 "B.Cu" signal)
-		(9 "F.Adhes" user)
-		(11 "B.Adhes" user)
+		(9 "F.Adhes" user "F.Adhesive")
+		(11 "B.Adhes" user "B.Adhesive")
 		(13 "F.Paste" user)
 		(15 "B.Paste" user)
-		(5 "F.SilkS" user)
-		(7 "B.SilkS" user)
+		(5 "F.SilkS" user "F.Silkscreen")
+		(7 "B.SilkS" user "B.Silkscreen")
 		(1 "F.Mask" user)
 		(3 "B.Mask" user)
-		(17 "Dwgs.User" user)
-		(19 "Cmts.User" user)
-		(21 "Eco1.User" user)
-		(23 "Eco2.User" user)
+		(17 "Dwgs.User" user "User.Drawings")
+		(19 "Cmts.User" user "User.Comments")
+		(21 "Eco1.User" user "User.Eco1")
+		(23 "Eco2.User" user "User.Eco2")
 		(25 "Edge.Cuts" user)
 		(27 "Margin" user)
-		(31 "F.CrtYd" user)
-		(29 "B.CrtYd" user)
+		(31 "F.CrtYd" user "F.Courtyard")
+		(29 "B.CrtYd" user "B.Courtyard")
 		(35 "F.Fab" user)
 		(33 "B.Fab" user)
@@
 		)
 	)
-	(footprint "Capacitor_SMD:C_0201_0603Metric"
+	(footprint "Capacitor_SMD:C_0402_1005Metric"
 		(layer "F.Cu")
-		(at 145.8251 115.66526 90)
-		(descr "Capacitor SMD 0201 (0603 Metric), square (rectangular) end terminal, IPC-7351 nominal, (Body size source: https://www.vishay.com/docs/20052/crcw0201e3.pdf), generated with kicad-footprint-generator")
+		(at 145.8251 115.82026 90)
+		(descr "Capacitor SMD 0402 (1005 Metric), square (rectangular) end terminal, IPC-7351 nominal, (Body size source: IPC-SM-782 page 76, https://www.pcb-3d.com/wordpress/wp-content/uploads/ipc-sm-782a_amendment_1_and_2.pdf), generated with kicad-footprint-generator")
 		(tags "capacitor")
 		(property "Reference" "C10"
-			(at 0 0 90)
+			(at 0 -1.16 90)
 			(layer "F.SilkS")
 			(hide yes)
 			(effects
 				(font
-					(size 0.2 0.2)
-					(thickness 0.05)
-					(bold yes)
+					(size 1 1)
+					(thickness 0.15)
 				)
 			)
 		)
 		(property "Value" "10n"
-			(at 0 1.05 90)
+			(at 0 1.16 90)
 			(layer "F.Fab")
 			(hide yes)
@@
 			(effects
 				(font
-					(size 0.2 1.27)
-					(thickness 0.05)
+					(size 1.27 1.27)
+					(thickness 0.15)
 				)
 			)
@@
 			(effects
 				(font
-					(size 0.2 1.27)
-					(thickness 0.05)
+					(size 1.27 1.27)
+					(thickness 0.15)
 				)
 			)
@@
 		(attr smd)
 		(fp_line
-			(start 0.7 -0.35)
-			(end 0.7 0.35)
+			(start -0.107836 -0.36)
+			(end 0.107836 -0.36)
+			(stroke
+				(width 0.12)
+				(type solid)
+			)
+			(layer "F.SilkS")
+		)
+		(fp_line
+			(start -0.107836 0.36)
+			(end 0.107836 0.36)
+			(stroke
+				(width 0.12)
+				(type solid)
+			)
+			(layer "F.SilkS")
+		)
+		(fp_line
+			(start 0.91 -0.46)
+			(end 0.91 0.46)
 			(stroke
 				(width 0.05)
@@
 		)
 		(fp_line
-			(start -0.7 -0.35)
-			(end 0.7 -0.35)
+			(start -0.91 -0.46)
+			(end 0.91 -0.46)
 			(stroke
 				(width 0.05)
@@
 		)
 		(fp_line
-			(start 0.7 0.35)
-			(end -0.7 0.35)
+			(start 0.91 0.46)
+			(end -0.91 0.46)
 			(stroke
 				(width 0.05)
@@
 		)
 		(fp_line
-			(start -0.7 0.35)
-			(end -0.7 -0.35)
+			(start -0.91 0.46)
+			(end -0.91 -0.46)
 			(stroke
 				(width 0.05)
@@
 		)
 		(fp_line
-			(start 0.3 -0.15)
-			(end 0.3 0.15)
+			(start 0.5 -0.25)
+			(end 0.5 0.25)
 			(stroke
 				(width 0.1)
@@
 		)
 		(fp_line
-			(start -0.3 -0.15)
-			(end 0.3 -0.15)
+			(start -0.5 -0.25)
+			(end 0.5 -0.25)
 			(stroke
 				(width 0.1)
@@
 		)
 		(fp_line
-			(start 0.3 0.15)
-			(end -0.3 0.15)
+			(start 0.5 0.25)
+			(end -0.5 0.25)
 			(stroke
 				(width 0.1)
@@
 		)
 		(fp_line
-			(start -0.3 0.15)
-			(end -0.3 -0.15)
+			(start -0.5 0.25)
+			(end -0.5 -0.25)
 			(stroke
 				(width 0.1)
@@
 		)
 		(fp_text user "${REFERENCE}"
-			(at -0.675 0.905 0)
+			(at 0 0 90)
 			(layer "F.Fab")
 			(effects
 				(font
-					(size 0.2 0.2)
+					(size 0.25 0.25)
 					(thickness 0.04)
 				)
 			)
 		)
-		(pad "" smd roundrect
-			(at -0.345 0 90)
-			(size 0.318 0.36)
-			(layers "F.Paste")
-			(roundrect_rratio 0.25)
-		)
-		(pad "" smd roundrect
-			(at 0.345 0 90)
-			(size 0.318 0.36)
-			(layers "F.Paste")
-			(roundrect_rratio 0.25)
-		)
 		(pad "1" smd roundrect
-			(at -0.32 0 90)
-			(size 0.46 0.4)
-			(layers "F.Cu" "F.Mask")
+			(at -0.48 0 90)
+			(size 0.56 0.62)
+			(layers "F.Cu" "F.Mask" "F.Paste")
 			(roundrect_rratio 0.25)
 			(net 1 "+3.3V")
@@
 		)
 		(pad "2" smd roundrect
-			(at 0.32 0 90)
-			(size 0.46 0.4)
-			(layers "F.Cu" "F.Mask")
+			(at 0.48 0 90)
+			(size 0.56 0.62)
+			(layers "F.Cu" "F.Mask" "F.Paste")
 			(roundrect_rratio 0.25)
 			(net 2 "GND")
@@
 		)
 		(embedded_fonts no)
-		(model "${KICAD9_3DMODEL_DIR}/Capacitor_SMD.3dshapes/C_0201_0603Metric.step"
+		(model "${KICAD9_3DMODEL_DIR}/Capacitor_SMD.3dshapes/C_0402_1005Metric.step"
 			(offset
 				(xyz 0 0 0)
@@
 	)
 	(segment
+		(start 145.5101 115.98526)
+		(end 145.8251 116.30026)
+		(width 0.25)
+		(layer "F.Cu")
+		(net 1)
+	)
+	(segment
 		(start 133.0511 96.64526)
 		(end 133.0511 95.89526)
@@
 	)
 	(segment
+		(start 144.7161 115.98526)
+		(end 145.5101 115.98526)
+		(width 0.25)
+		(layer "F.Cu")
+		(net 1)
+	)
+	(segment
 		(start 129.5511 99.92026)
 		(end 129.5761 99.89526)
@@
 	)
 	(segment
+		(start 146.5511 116.32026)
+		(end 146.0001 116.32026)
+		(width 0.25)
+		(layer "F.Cu")
+		(net 1)
+	)
+	(segment
 		(start 135.5311 110.82026)
 		(end 135.5311 111.80026)
@@
 	)
 	(segment
-		(start 145.8251 115.98526)
-		(end 144.7161 115.98526)
-		(width 0.25)
-		(layer "F.Cu")
-		(net 1)
-	)
-	(segment
 		(start 132.8111 90.49026)
 		(end 132.8111 89.42026)
@@
 	)
 	(segment
-		(start 145.8251 115.98526)
-		(end 145.8251 116.48526)
-		(width 0.25)
+		(start 154.0511 106.32026)
+		(end 153.6461 106.72526)
+		(width 0.5)
 		(layer "F.Cu")
 		(net 1)
 	)
 	(segment
-		(start 154.0511 106.32026)
-		(end 153.6461 106.72526)
-		(width 0.5)
+		(start 146.0001 116.32026)
+		(end 145.8251 116.14526)
+		(width 0.25)
 		(layer "F.Cu")
 		(net 1)
@@
 	)
 	(via
-		(at 145.8251 116.48526)
+		(at 146.5511 116.32026)
 		(size 0.8)
 		(drill 0.4)
@@
 	)
 	(segment
-		(start 146.5261 115.34526)
-		(end 146.6511 115.22026)
-		(width 0.25)
-		(layer "F.Cu")
-		(net 2)
-	)
-	(segment
 		(start 158.3761 113.53026)
 		(end 158.3761 115.45526)
@@
 	)
 	(segment
+		(start 145.8251 115.34026)
+		(end 146.5311 115.34026)
+		(width 0.25)
+		(layer "F.Cu")
+		(net 2)
+	)
+	(segment
 		(start 128.9311 94.30026)
 		(end 129.3361 93.89526)
@@
 	)
 	(segment
-		(start 145.8251 115.34526)
-		(end 146.5261 115.34526)
-		(width 0.25)
-		(layer "F.Cu")
-		(net 2)
-	)
-	(segment
 		(start 127.8611 91.76026)
 		(end 128.9711 91.76026)
@@
 	)
 	(segment
+		(start 146.5311 115.34026)
+		(end 146.6511 115.22026)
+		(width 0.25)
+		(layer "F.Cu")
+		(net 2)
+	)
+	(segment
 		(start 126.7411 94.30026)
 		(end 126.3361 93.89526)
@@
 	)
 	(via
+		(at 149.5511 110.82026)
+		(size 0.8)
+		(drill 0.4)
+		(layers "F.Cu" "B.Cu")
+		(net 2)
+	)
+	(via
 		(at 124.0511 113.89526)
 		(size 0.8)
@@
 	)
 	(via
+		(at 154.5511 108.82026)
+		(size 0.8)
+		(drill 0.4)
+		(layers "F.Cu" "B.Cu")
+		(net 2)
+	)
+	(via
 		(at 149.0511 98.82026)
 		(size 0.8)
@@
 	)
 	(via
+		(at 151.0511 110.82026)
+		(size 0.8)
+		(drill 0.4)
+		(layers "F.Cu" "B.Cu")
+		(net 2)
+	)
+	(via
 		(at 129.3361 91.39526)
 		(size 0.8)
@@
 	)
 	(via
+		(at 154.0511 110.82026)
+		(size 0.8)
+		(drill 0.4)
+		(layers "F.Cu" "B.Cu")
+		(net 2)
+	)
+	(via
 		(at 126.5261 110.14526)
 		(size 0.8)
@@
 	)
 	(via
+		(at 152.5511 108.82026)
+		(size 0.8)
+		(drill 0.4)
+		(layers "F.Cu" "B.Cu")
+		(net 2)
+	)
+	(via
 		(at 123.5511 115.32026)
 		(size 0.8)
@@
 	)
 	(via
+		(at 155.5511 110.82026)
+		(size 0.8)
+		(drill 0.4)
+		(layers "F.Cu" "B.Cu")
+		(net 2)
+	)
+	(via
 		(at 132.5511 115.32026)
 		(size 0.8)
@@
 	)
 	(via
+		(at 156.5511 108.82026)
+		(size 0.8)
+		(drill 0.4)
+		(layers "F.Cu" "B.Cu")
+		(net 2)
+	)
+	(via
 		(at 124.7011 104.89526)
 		(size 0.8)
@@
 	)
 	(via
+		(at 152.5511 110.82026)
+		(size 0.8)
+		(drill 0.4)
+		(layers "F.Cu" "B.Cu")
+		(net 2)
+	)
+	(via
 		(at 129.5761 110.14526)
 		(size 0.8)
@@
 		(size 0.8)
 		(drill 0.4)
+		(layers "F.Cu" "B.Cu")
+		(net 2)
+	)
+	(via
+		(at 151.0511 108.82026)
+		(size 0.8)
+		(drill 0.4)
